File: circuit/RF_INPUT.brd (EAGLE design)
At the start: 64.4 x 80 mm, 98 parts, among them IC1 TS464, IC2 SN74LVC1G3157DBVR, Q1 IRML6302, Q2 IRML6302, Q3 2N7002, U1 SA612, U2 SA612, U3 SA612, X1 BU-SMA-V, X4 SMA-142-0701-801/806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

Commit message: - работающий в первом приближении USB Virtual Com Port
Parts:
- C18, C25, C4: value 220N -> 1u
- C20, C21, C31, C32, C7, C8: value 220N -> 2u2
- R10, R42: value 4.7k -> 5K4
- R23, R27: value 4K7 -> 3K9
- R28, R30: value 10K -> 9K1
- R35, R40: value 22K -> 3K9
- R4, R7: value 15K -> 3K9

Commit message: - начали рисовать платку с дифференциальным входом.
Parts:
- X4, X6: value SMA-142-0701-801/806 -> SMA
Changed lines of the file:
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@@
 <?xml version="1.0" encoding="utf-8"?>
 <!DOCTYPE eagle SYSTEM "eagle.dtd">
-<eagle version="7.1.0">
+<eagle version="7.4.0">
 <drawing>
 <settings>
@@
 <element name="U1" library="vnwa" package="SO8" value="SA612" x="15.24" y="33.655" rot="R180"/>
 <element name="U3" library="vnwa" package="SO8" value="SA612" x="24.13" y="12.065" rot="R270"/>
-<element name="X4" library="con-coax" package="J502-ND-142-0701-801/806" value="SMA-142-0701-801/806" x="1.27" y="69.85">
+<element name="X4" library="con-coax" package="J502-ND-142-0701-801/806" value="SMA" x="1.27" y="69.85">
 <attribute name="OC_NEWARK" value="90F2624" x="1.27" y="69.85" size="1.778" layer="27" display="off"/>
 <attribute name="MPN" value="142-0701-801" x="1.27" y="69.85" size="1.778" layer="27" display="off"/>
@@
 <attribute name="OC_FARNELL" value="1608592" x="1.27" y="69.85" size="1.778" layer="27" display="off"/>
 </element>
-<element name="X6" library="con-coax" package="J502-ND-142-0701-801/806" value="SMA-142-0701-801/806" x="1.27" y="10.16">
+<element name="X6" library="con-coax" package="J502-ND-142-0701-801/806" value="SMA" x="1.27" y="10.16">
 <attribute name="OC_NEWARK" value="90F2624" x="1.27" y="10.16" size="1.778" layer="27" display="off"/>
 <attribute name="MPN" value="142-0701-801" x="1.27" y="10.16" size="1.778" layer="27" display="off"/>
