File: circuit/RF_INPUT_DIFF.sch (EAGLE design)
At the start: 100 parts, among them IC1 TS464, IC4 TS462D, IC5 TS462D, IC6 TS462D, IC7 4052D, Q1 IRML6302, Q2 IRML6302, Q3 2N7002, U1 SA612, U2 SA612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

Commit message: - продолжили работу над diff входом
Parts:
- removed C30: nc, rcl:C-EUC0805
- removed C36: 100N, rcl:C-EUC0603
- removed C9: 100n, rcl:C-EUC0603
- removed IC7: 4052D, 40xx:4052D
- removed X4, X6: SMA, con-coax:SMA-142-0701-801/806
- added IC2: SN74LVC1G3157DBVR, balmer:SN74LVC1G3157DBVR
- added R49, R51: 220, rcl:R-EU_R0603
- added R50: 22K, rcl:R-EU_R0603
- added RX, TX: SMA, con-coax:SMA-142-0701-801/806
- added X2: (no value), con-phoenix-254:MPT6
- IC1: value TS464 -> SN74LVC1G3157DBVR; device linear:AD8684R -> balmer:SN74LVC1G3157DBVR
- R24: value 330K -> 4.7K
- R25, R26: value 4K7 -> 330K
- R39: value 22K -> 150K
- R41: value 330k -> 22K
- R5: value 330K -> 15K
- R6, R9: value 15K -> 330K
Connections:
- net ADC_REF_M renamed REF_B
- net ADC_REF_P renamed REF_A
- removed net ADC_SWITCH_NO: C30.1, IC1C.OUT, R37.2
- removed net N$41: C30.2, IC1C.-IN, R37.1, R38.2
- removed net N$43: C31.1, R38.1
- removed net N$44: C32.1, R39.1
- removed net N$46: IC1D.-IN, IC1D.OUT
- removed net N$47: IC1C.+IN, R39.2, R41.1
- new net N$11: C31.1, IC6A.+IN, R41.1
- new net N$12: C32.1, IC6B.+IN, R50.2
- new net N$2: IC6A.-IN, R37.1, R38.1
- new net N$25: IC6A.OUT, R37.2, R45.1
- new net N$26: IC6B.-IN, R38.2, R39.1
- new net N$27: IC6B.OUT, R39.2, R51.1
- new net RX_A: IC1.B2, R49.2
- new net RX_B: IC2.B2, R36.2
- new net TX_A: IC1.B1, R51.2
- new net TX_B: IC2.B1, R45.2
- net +6V0: now also IC1.VCC, IC2.VCC, IC4P.V+, IC5P.V+, IC6P.V+; no longer C9.1, IC1P.V+
- net GND: now also IC1.GND, IC2.GND, IC4P.V-, IC5P.V-, IC6P.V-, RX.2, TX.2; no longer C36.2, C9.2, IC1D.+IN, IC1P.V-, X4.2, X6.2
- net N$23: now also R36.1
- net N$24: now also R49.1
- net N$30: now also TX.1; no longer X6.1
- net N$5: now also RX.1; no longer X4.1
- net OPA_BIAS: now also R50.1; no longer C36.1
- net SET_CHANNEL: now also IC1.S, IC2.S
Other:
- note removed: "BRIDGE AND TRANSMITTER"
- note removed: "THRU RECEIVER AND MUX"
- moved on the sheet: C1, C10, C11, C12, C13, C14, C15, C16, C17, C18, C2, C20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

Commit message: - начали рисовать платку для diff выхода.
Parts:
- removed R36, R45, R46, R49, R51, R8: 220, rcl:R-EU_R0603
- C10, C11, C22, C23, C33, C34: value 1N -> 10N
Connections:
- removed net N$15: IC4A.OUT, R6.2, R8.2
- removed net N$16: IC4B.OUT, R46.2, R9.2
- removed net N$23: IC5A.OUT, R25.2, R36.1
- removed net N$24: IC5B.OUT, R26.2, R49.1
- removed net N$25: IC6A.OUT, R37.2, R45.1
- removed net N$27: IC6B.OUT, R39.2, R51.1
- new net ADC_A: IC1.A, X2-4.1
- new net ADC_B: IC2.A, X2-5.1
- net GND: now also X2-1.1, X2-6.1
- net REF_A: now also IC4A.OUT, R6.2, X2-3.1; no longer R8.1
- net REF_B: now also IC4B.OUT, R9.2, X2-2.1; no longer R46.1
- net RX_A: now also IC5B.OUT, R26.2; no longer R49.2
- net RX_B: now also IC5A.OUT, R25.2; no longer R36.2
- net TX_A: now also IC6B.OUT, R39.2; no longer R51.2
- net TX_B: now also IC6A.OUT, R37.2; no longer R45.2
Other:
- moved on the sheet: IC1, IC2, X2-1, X2-2, X2-3, X2-4, X2-5, X2-6

Commit message: - начали калибровку по S параметрам
Connections:
- net +6V0: no longer IC5P.V+, IC6P.V+
- net N$4: now also IC6P.V+
- net N$8: now also IC5P.V+
Changed lines of the file:
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@@
 <wire x1="121.92" y1="91.44" x2="132.08" y2="91.44" width="0.1524" layer="91"/>
 <junction x="132.08" y="91.44"/>
-<pinref part="IC6" gate="P" pin="V+"/>
-<wire x1="132.08" y1="106.68" x2="139.7" y2="106.68" width="0.1524" layer="91"/>
 </segment>
 <segment>
@@
 <wire x1="83.82" y1="210.82" x2="96.52" y2="210.82" width="0.1524" layer="91"/>
 <junction x="96.52" y="210.82"/>
-<pinref part="IC5" gate="P" pin="V+"/>
-<wire x1="104.14" y1="223.52" x2="96.52" y2="223.52" width="0.1524" layer="91"/>
-<junction x="96.52" y="223.52"/>
 </segment>
 <segment>
@@
 <wire x1="167.64" y1="73.66" x2="157.48" y2="73.66" width="0.1524" layer="91"/>
 <pinref part="Q2" gate="G$1" pin="D"/>
-<wire x1="149.86" y1="73.66" x2="132.08" y2="73.66" width="0.1524" layer="91"/>
+<wire x1="149.86" y1="73.66" x2="144.78" y2="73.66" width="0.1524" layer="91"/>
 <junction x="149.86" y="73.66"/>
 <junction x="157.48" y="73.66"/>
+<pinref part="IC6" gate="P" pin="V+"/>
+<wire x1="142.24" y1="73.66" x2="132.08" y2="73.66" width="0.1524" layer="91"/>
+<wire x1="139.7" y1="106.68" x2="142.24" y2="106.68" width="0.1524" layer="91"/>
+<wire x1="142.24" y1="106.68" x2="142.24" y2="73.66" width="0.1524" layer="91"/>
+<wire x1="142.24" y1="73.66" x2="144.78" y2="73.66" width="0.1524" layer="91"/>
+<junction x="142.24" y="73.66"/>
 </segment>
 </net>
@@
 <junction x="124.46" y="193.04"/>
 <pinref part="Q1" gate="G$1" pin="D"/>
-<wire x1="119.38" y1="193.04" x2="96.52" y2="193.04" width="0.1524" layer="91"/>
+<wire x1="119.38" y1="193.04" x2="109.22" y2="193.04" width="0.1524" layer="91"/>
 <junction x="119.38" y="193.04"/>
+<pinref part="IC5" gate="P" pin="V+"/>
+<wire x1="109.22" y1="193.04" x2="96.52" y2="193.04" width="0.1524" layer="91"/>
+<wire x1="104.14" y1="223.52" x2="109.22" y2="223.52" width="0.1524" layer="91"/>
+<wire x1="109.22" y1="223.52" x2="109.22" y2="193.04" width="0.1524" layer="91"/>
+<junction x="109.22" y="193.04"/>
 </segment>
 </net>
